File: cc2652r_v2_rs.brd (EAGLE design)
At the start: 29.3 x 29.3 mm, 55 parts, among them IC3 CC2652R1FRGZ, SW1 MOMENTARY-SWITCH-SPST-SMD-4.6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, Y1 Q22FA12800150, Y2 32.768KHz

Commit message: Add files via upload
Parts:
- turned SW1 to 180 degrees
Routing:
- net GND: track 25.4 -> 23.1 mm, vias 254 -> 275
- net N$6: track 30.3 -> 32.1 mm

Commit message: Add files via upload
Parts:
- added C26: CAP0402, discretes-dev:CAPC1005X40N
- moved C21 3.87 mm to (22.8, 20.7)
- moved C19 3.69 mm to (21.8, 18.7), turned to 63 degrees
- moved L6 0.55 mm to (20.5, 13.2), turned to 89.4 degrees
Connections:
- net GND: now also C26.1
- net N$9: now also C26.2
Routing:
- net N$5: track 1.24 -> 4.78 mm
- net N$9: track 5.14 -> 2.22 mm
- net GND: vias 275 -> 268
