File: cc2652r_v2_rs.brd (EAGLE design)
At the start: 29.3 x 29.3 mm, 56 parts, among them IC3 CC2652R1FRGZ, SW1 MOMENTARY-SWITCH-SPST-SMD-4.6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, Y1 Q22FA12800150, Y2 32.768KHz

Commit message: Add files via upload
Parts:
- removed C20, C22: CAP0402, discretes-dev:CAPC1005X40N
- moved R3 0.20 mm to (11.8, 4.20), turned to 180 degrees
Connections:
- net 2: now also R3.1, REEDSWITCH.1; no longer R3.2, REEDSWITCH.2
- net GND: now also REEDSWITCH.2; no longer C20.1, C22.2, R3.1
- net VCC: now also R3.2; no longer REEDSWITCH.1
- net X48M_N: no longer C22.1
- net X48M_P: no longer C20.2
Routing:
- net 2: track 25.6 -> 19.5 mm
- net VCC: track 65.8 -> 63.4 mm, vias 8 -> 9
- net GND: track 23.1 -> 25.0 mm, vias 271 -> 270
- net X48M_N: track 4.43 -> 2.62 mm
- net X48M_P: track 6.12 -> 4.94 mm

Commit message: Add files via upload
Routing:
- net 23: track 0.94 -> 0.00 mm, vias 1 -> 0
- net GND: vias 270 -> 303
Changed lines of the file:
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@@
 <drawing>
 <settings>
-<setting alwaysvectorfont="yes"/>
+<setting alwaysvectorfont="no"/>
 <setting verticaltext="up"/>
 </settings>
@@
 <wire x1="21.844" y1="17.526" x2="23.622" y2="21.082" width="0.254" layer="41"/>
 <wire x1="23.622" y1="21.082" x2="24.003" y2="21.336" width="0.254" layer="41" curve="-59.489763"/>
-<wire x1="23.622" y1="22.225" x2="22.987" y2="21.717" width="0.254" layer="41" curve="61.927586"/>
-<wire x1="23.622" y1="22.225" x2="24.003" y2="22.225" width="0.254" layer="41"/>
+<wire x1="23.749" y1="22.225" x2="22.987" y2="21.717" width="0.254" layer="41" curve="61.927586"/>
+<wire x1="23.749" y1="22.225" x2="24.13" y2="22.225" width="0.254" layer="41"/>
 <wire x1="22.86" y1="21.5138" x2="23.0251" y2="21.8186" width="0.254" layer="41"/>
 <wire x1="23.4188" y1="24.511" x2="24.0665" y2="24.511" width="0.2" layer="41"/>
 <wire x1="23.4188" y1="23.2791" x2="24.0665" y2="23.2791" width="0.2" layer="41"/>
 <wire x1="23.4188" y1="24.511" x2="23.4188" y2="23.2791" width="0.2" layer="41"/>
+<wire x1="18.796" y1="12.319" x2="19.939" y2="12.319" width="0.254" layer="41"/>
+<wire x1="18.796" y1="11.176" x2="19.939" y2="11.176" width="0.254" layer="41"/>
+<wire x1="20.066" y1="11.176" x2="19.939" y2="11.176" width="0.254" layer="41"/>
+<wire x1="20.066" y1="11.176" x2="21.209" y2="11.176" width="0.254" layer="41"/>
 </plain>
 <attributes>
@@
 <wire x1="8.0816" y1="12.101" x2="8.0618" y2="12.0812" width="0.1524" layer="1"/>
 <wire x1="8.0618" y1="12.0812" x2="7.4279" y2="12.0812" width="0.1524" layer="1"/>
-<wire x1="7.4279" y1="12.0812" x2="6.9507" y2="11.604" width="0.1524" layer="1"/>
-<wire x1="6.9507" y1="11.604" x2="6.9507" y2="10.9055" width="0.1524" layer="1"/>
+<wire x1="7.4279" y1="12.0812" x2="7.2047" y2="11.858" width="0.1524" layer="1"/>
+<wire x1="7.2047" y1="11.858" x2="7.2047" y2="10.6515" width="0.1524" layer="1"/>
 <via x="8.3693" y="9.7663" extent="1-16" drill="0.2" diameter="0.45"/>
-<wire x1="6.9507" y1="10.9055" x2="8.0899" y2="9.7663" width="0.1524" layer="1"/>
+<wire x1="7.2047" y1="10.6515" x2="8.0899" y2="9.7663" width="0.1524" layer="1"/>
 <wire x1="8.0899" y1="9.7663" x2="8.3693" y2="9.7663" width="0.1524" layer="1"/>
 <wire x1="8.3693" y1="9.7663" x2="8.3693" y2="9.7409" width="0.1524" layer="1"/>
@@
 <via x="21.971" y="22.9362" extent="1-16" drill="0.25"/>
 <via x="22.606" y="22.9362" extent="1-16" drill="0.25"/>
-<via x="22.098" y="12.827" extent="1-16" drill="0.25"/>
-<via x="21.463" y="12.827" extent="1-16" drill="0.25"/>
+<via x="22.098" y="12.7" extent="1-16" drill="0.25"/>
+<via x="21.463" y="12.7" extent="1-16" drill="0.25"/>
 <via x="21.463" y="13.589" extent="1-16" drill="0.25"/>
 <via x="21.463" y="14.351" extent="1-16" drill="0.25"/>
@@
 <via x="15.4559" y="6.7818" extent="1-16" drill="0.254"/>
 <via x="12.192" y="3.429" extent="1-16" drill="0.25"/>
+<via x="23.241" y="11.811" extent="1-16" drill="0.25"/>
+<via x="23.241" y="12.446" extent="1-16" drill="0.25"/>
+<via x="23.241" y="13.081" extent="1-16" drill="0.25"/>
+<via x="23.241" y="13.716" extent="1-16" drill="0.25"/>
+<via x="23.241" y="14.351" extent="1-16" drill="0.25"/>
+<via x="23.241" y="14.986" extent="1-16" drill="0.25"/>
+<via x="23.241" y="15.621" extent="1-16" drill="0.25"/>
+<via x="23.241" y="16.256" extent="1-16" drill="0.25"/>
+<via x="23.241" y="16.891" extent="1-16" drill="0.25"/>
+<via x="23.241" y="17.526" extent="1-16" drill="0.25"/>
+<via x="23.241" y="18.161" extent="1-16" drill="0.25"/>
+<via x="22.606" y="13.081" extent="1-16" drill="0.25"/>
+<via x="22.606" y="13.716" extent="1-16" drill="0.25"/>
+<via x="22.606" y="14.351" extent="1-16" drill="0.25"/>
+<via x="22.606" y="14.986" extent="1-16" drill="0.25"/>
+<via x="22.606" y="15.621" extent="1-16" drill="0.25"/>
+<via x="22.606" y="16.256" extent="1-16" drill="0.25"/>
+<via x="22.606" y="16.891" extent="1-16" drill="0.25"/>
+<via x="22.606" y="25.527" extent="1-16" drill="0.25"/>
+<via x="22.606" y="26.162" extent="1-16" drill="0.25"/>
+<via x="22.606" y="26.797" extent="1-16" drill="0.25"/>
+<via x="22.606" y="27.432" extent="1-16" drill="0.25"/>
+<via x="20.701" y="9.271" extent="1-16" drill="0.25"/>
+<via x="20.701" y="8.636" extent="1-16" drill="0.25"/>
+<via x="21.336" y="8.636" extent="1-16" drill="0.25"/>
+<via x="21.971" y="8.636" extent="1-16" drill="0.25"/>
+<via x="22.606" y="8.636" extent="1-16" drill="0.25"/>
+<via x="22.606" y="9.271" extent="1-16" drill="0.25"/>
+<via x="21.971" y="9.271" extent="1-16" drill="0.25"/>
+<via x="21.336" y="9.271" extent="1-16" drill="0.25"/>
+<via x="8.001" y="10.795" extent="1-16" drill="0.25"/>
+<via x="9.017" y="9.906" extent="1-16" drill="0.25"/>
+<via x="10.541" y="9.779" extent="1-16" drill="0.25"/>
 </signal>
 <signal name="DCOUPL">
@@
 <wire x1="14.9816" y1="14.601" x2="15.8155" y2="14.601" width="0.1524" layer="1"/>
 <wire x1="15.8155" y1="14.601" x2="16.1036" y2="14.3129" width="0.1524" layer="1"/>
-<via x="16.1036" y="14.3129" extent="1-16" drill="0.25"/>
+<via x="16.1036" y="14.3129" extent="1-16" drill="0.2" diameter="0.45"/>
 <wire x1="16.1036" y1="14.3129" x2="15.8496" y2="14.0589" width="0.1524" layer="2"/>
 <wire x1="15.8496" y1="14.0589" x2="15.8496" y2="11.9775375" width="0.1524" layer="2"/>
@@
 <wire x1="14.9816" y1="15.601" x2="15.768" y2="15.601" width="0.1524" layer="1"/>
 <wire x1="15.768" y1="15.601" x2="15.875" y2="15.494" width="0.1524" layer="1"/>
-<via x="15.875" y="15.494" extent="1-16" drill="0.25"/>
+<via x="15.875" y="15.494" extent="1-16" drill="0.2" diameter="0.45"/>
 <wire x1="3.556" y1="3.8481" x2="6.6441" y2="6.9362" width="0.1524" layer="2"/>
 <wire x1="6.6441" y1="6.9362" x2="6.65503125" y2="6.9362" width="0.1524" layer="2"/>
@@
 <wire x1="14.9816" y1="16.101" x2="15.847" y2="16.101" width="0.1524" layer="1"/>
 <wire x1="15.847" y1="16.101" x2="15.875" y2="16.129" width="0.1524" layer="1"/>
-<via x="15.875" y="16.129" extent="1-16" drill="0.25"/>
+<via x="15.875" y="16.129" extent="1-16" drill="0.2" diameter="0.45"/>
 <wire x1="4.2037" y1="3.8735" x2="4.2037" y2="4.1006625" width="0.1524" layer="2"/>
 <wire x1="6.7598375" y1="6.6568" x2="6.77076875" y2="6.6568" width="0.1524" layer="2"/>
@@
 <signal name="23">
 <contactref element="IC3" pad="36"/>
-<wire x1="8.0816" y1="11.601" x2="7.6259" y2="11.601" width="0.1524" layer="1"/>
-<wire x1="7.6259" y1="11.601" x2="7.4295" y2="11.4046" width="0.1524" layer="1"/>
-<wire x1="7.4295" y1="11.4046" x2="7.4295" y2="11.2522" width="0.1524" layer="1"/>
-<wire x1="7.4295" y1="11.2522" x2="7.3914" y2="11.2141" width="0.1524" layer="1"/>
-<via x="7.3914" y="11.2141" extent="1-16" drill="0.2" diameter="0.45"/>
 </signal>
 <signal name="24">

Commit message: Add files via upload
Connections:
- net 11: now also BME280.2, BME280.6, BME280.8, C24.2, C25.1, HTU21.5
- net VCC: no longer BME280.2, BME280.6, BME280.8, C24.2, C25.1, HTU21.5
Routing:
- net 11: track 0.00 -> 42.9 mm, vias 0 -> 3
- net VCC: track 63.4 -> 44.7 mm, vias 9 -> 6
- net N$6: track 32.1 -> 30.8 mm
- net 7: track 16.6 -> 15.4 mm

Commit message: Add files via upload
Routing:
- net 11: track 42.9 -> 46.8 mm
- net GND: vias 303 -> 321
Other:
- outline, holes or cut-outs redrawn
Changed lines of the file:
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@@
 </polygon>
 <text x="0.92480625" y="4.10315625" size="0.8128" layer="26" rot="MR90">JLCJLCJLCJLC</text>
-<wire x1="9.6397625" y1="0.997396875" x2="9.6397625" y2="-0.102603125" width="0.0762" layer="20"/>
-<wire x1="9.6397625" y1="-0.102603125" x2="25.9667625" y2="-0.102603125" width="0.0762" layer="20"/>
+<wire x1="9.5127625" y1="0.997396875" x2="9.5127625" y2="-0.102603125" width="0.0762" layer="20"/>
+<wire x1="9.5127625" y1="-0.102603125" x2="25.9667625" y2="-0.102603125" width="0.0762" layer="20"/>
 <wire x1="25.9667625" y1="-0.102603125" x2="25.9667625" y2="2.097396875" width="0.0762" layer="20"/>
 <wire x1="27.2667625" y1="3.297396875" x2="29.3667625" y2="3.297396875" width="0.0762" layer="20"/>
@@
 <wire x1="29.3667625" y1="22.297396875" x2="29.3667625" y2="25.797396875" width="0.0762" layer="20"/>
 <wire x1="29.3667625" y1="25.797396875" x2="27.1667625" y2="25.797396875" width="0.0762" layer="20"/>
-<wire x1="9.6397625" y1="0.997396875" x2="8.8397625" y2="0.997396875" width="0.0762" layer="20"/>
-<wire x1="8.8397625" y1="0.997396875" x2="8.8397625" y2="-0.102603125" width="0.0762" layer="20"/>
-<wire x1="8.8397625" y1="-0.102603125" x2="3.4667625" y2="-0.102603125" width="0.0762" layer="20"/>
+<wire x1="9.5127625" y1="0.997396875" x2="8.5857625" y2="0.997396875" width="0.0762" layer="20"/>
+<wire x1="8.5857625" y1="0.997396875" x2="8.5857625" y2="-0.102603125" width="0.0762" layer="20"/>
+<wire x1="8.5857625" y1="-0.102603125" x2="3.4667625" y2="-0.102603125" width="0.0762" layer="20"/>
 <wire x1="3.4667625" y1="-0.102603125" x2="3.4667625" y2="1.897396875" width="0.0762" layer="20"/>
 <wire x1="0.0667625" y1="3.397396875" x2="2.1667625" y2="3.397396875" width="0.0762" layer="20"/>
@@
 <wire x1="0.0667625" y1="25.797396875" x2="2.3667625" y2="25.797396875" width="0.0762" layer="20"/>
 <wire x1="3.6667625" y1="29.197396875" x2="3.6667625" y2="27.097396875" width="0.0762" layer="20"/>
-<wire x1="3.6667625" y1="29.197396875" x2="8.8397625" y2="29.197396875" width="0.0762" layer="20"/>
-<wire x1="8.8397625" y1="29.197396875" x2="8.8397625" y2="28.070396875" width="0.0762" layer="20"/>
-<wire x1="8.8397625" y1="28.070396875" x2="9.5397625" y2="28.070396875" width="0.0762" layer="20"/>
+<wire x1="3.6667625" y1="29.197396875" x2="8.5857625" y2="29.197396875" width="0.0762" layer="20"/>
+<wire x1="8.5857625" y1="29.197396875" x2="8.5857625" y2="28.070396875" width="0.0762" layer="20"/>
+<wire x1="8.5857625" y1="28.070396875" x2="9.5397625" y2="28.070396875" width="0.0762" layer="20"/>
 <wire x1="9.5397625" y1="28.070396875" x2="9.5397625" y2="29.197396875" width="0.0762" layer="20"/>
 <wire x1="9.5397625" y1="29.197396875" x2="26.0667625" y2="29.197396875" width="0.0762" layer="20"/>
@@
 <wire x1="21.082" y1="12.446" x2="21.082" y2="14.097" width="0.254" layer="41"/>
 <wire x1="21.082" y1="14.097" x2="21.844" y2="17.526" width="0.254" layer="41" curve="-25.057615"/>
-<wire x1="21.844" y1="17.526" x2="23.622" y2="21.082" width="0.254" layer="41"/>
-<wire x1="23.622" y1="21.082" x2="24.003" y2="21.336" width="0.254" layer="41" curve="-59.489763"/>
-<wire x1="23.749" y1="22.225" x2="22.987" y2="21.717" width="0.254" layer="41" curve="61.927586"/>
-<wire x1="23.749" y1="22.225" x2="24.13" y2="22.225" width="0.254" layer="41"/>
-<wire x1="22.86" y1="21.5138" x2="23.0251" y2="21.8186" width="0.254" layer="41"/>
+<wire x1="21.844" y1="17.526" x2="23.495" y2="20.955" width="0.254" layer="41"/>
+<wire x1="23.495" y1="20.955" x2="23.876" y2="21.209" width="0.254" layer="41" curve="-59.489763"/>
+<wire x1="23.495" y1="22.352" x2="22.86" y2="21.717" width="0.254" layer="41" curve="61.927586"/>
+<wire x1="23.495" y1="22.352" x2="24.003" y2="22.352" width="0.254" layer="41"/>
+<wire x1="22.733" y1="21.5138" x2="22.8981" y2="21.8186" width="0.254" layer="41"/>
 <wire x1="23.4188" y1="24.511" x2="24.0665" y2="24.511" width="0.2" layer="41"/>
 <wire x1="23.4188" y1="23.2791" x2="24.0665" y2="23.2791" width="0.2" layer="41"/>
 <wire x1="23.4188" y1="24.511" x2="23.4188" y2="23.2791" width="0.2" layer="41"/>
 <wire x1="18.796" y1="12.319" x2="19.939" y2="12.319" width="0.254" layer="41"/>
-<wire x1="18.796" y1="11.176" x2="19.939" y2="11.176" width="0.254" layer="41"/>
-<wire x1="20.066" y1="11.176" x2="19.939" y2="11.176" width="0.254" layer="41"/>
-<wire x1="20.066" y1="11.176" x2="21.209" y2="11.176" width="0.254" layer="41"/>
+<wire x1="18.796" y1="11.176" x2="21.209" y2="11.176" width="0.254" layer="41"/>
 </plain>
 <attributes>
@@
 <via x="11.176" y="28.702" extent="1-16" drill="0.25"/>
 <via x="10.541" y="28.702" extent="1-16" drill="0.25"/>
-<via x="8.255" y="28.702" extent="1-16" drill="0.25"/>
 <via x="7.493" y="28.702" extent="1-16" drill="0.25"/>
 <via x="6.731" y="28.702" extent="1-16" drill="0.25"/>
@@
 <via x="19.7612" y="19.8882" extent="1-16" drill="0.25"/>
 <via x="23.2537" y="22.9362" extent="1-16" drill="0.25"/>
-<via x="20.574" y="5.461" extent="1-16" drill="0.25"/>
 <via x="13.208" y="4.953" extent="1-16" drill="0.25"/>
 <via x="1.651" y="24.384" extent="1-16" drill="0.25"/>
@@
 <via x="9.017" y="9.906" extent="1-16" drill="0.25"/>
 <via x="10.541" y="9.779" extent="1-16" drill="0.25"/>
+<via x="18.415" y="15.367" extent="1-16" drill="0.25"/>
+<via x="18.415" y="16.002" extent="1-16" drill="0.25"/>
+<via x="19.05" y="15.748" extent="1-16" drill="0.25"/>
+<via x="19.177" y="16.51" extent="1-16" drill="0.25"/>
+<via x="19.05" y="14.986" extent="1-16" drill="0.25"/>
+<via x="21.971" y="13.97" extent="1-16" drill="0.25"/>
+<via x="22.098" y="14.605" extent="1-16" drill="0.25"/>
+<via x="22.098" y="15.24" extent="1-16" drill="0.25"/>
+<via x="18.161" y="6.096" extent="1-16" drill="0.25"/>
+<via x="18.161" y="5.461" extent="1-16" drill="0.25"/>
+<via x="18.796" y="6.096" extent="1-16" drill="0.25"/>
+<via x="19.431" y="6.096" extent="1-16" drill="0.25"/>
+<via x="20.066" y="6.096" extent="1-16" drill="0.25"/>
+<via x="18.796" y="5.461" extent="1-16" drill="0.25"/>
+<via x="19.431" y="5.461" extent="1-16" drill="0.25"/>
+<via x="20.066" y="5.461" extent="1-16" drill="0.25"/>
+<via x="20.701" y="5.461" extent="1-16" drill="0.25"/>
+<via x="21.336" y="23.5712" extent="1-16" drill="0.25"/>
+<via x="19.5326" y="20.9423" extent="1-16" drill="0.25"/>
+<via x="19.9136" y="21.7043" extent="1-16" drill="0.25"/>
 </signal>
 <signal name="DCOUPL">
@@
 <wire x1="5.9384" y1="4.0316" x2="5.9581" y2="4.0513" width="0.1524" layer="1"/>
 <wire x1="5.9384" y1="3.4873" x2="5.9384" y2="4.0316" width="0.1524" layer="1"/>
-<wire x1="6.2178" y1="0.7784" x2="6.2178" y2="0.3758" width="0.1524" layer="1"/>
-<wire x1="6.2178" y1="0.3758" x2="6.096" y2="0.254" width="0.1524" layer="1"/>
-<wire x1="6.096" y1="0.254" x2="4.445" y2="0.254" width="0.1524" layer="1"/>
-<wire x1="4.445" y1="0.254" x2="4.191" y2="0.508" width="0.1524" layer="1"/>
+<wire x1="4.191" y1="0.508" x2="4.445" y2="0.254" width="0.1524" layer="1"/>
 <via x="4.191" y="0.508" extent="1-16" drill="0.25"/>
 <wire x1="4.191" y1="0.508" x2="3.75446875" y2="0.94453125" width="0.1524" layer="2"/>
@@
 <wire x1="12.2816" y1="17.801" x2="12.2816" y2="18.6316" width="0.1524" layer="1"/>
 <wire x1="12.2816" y1="18.6316" x2="12.319" y2="18.669" width="0.1524" layer="1"/>
-<wire x1="5.5678" y1="2.8284" x2="6.8678" y2="2.8284" width="0" layer="19" extent="1-1"/>
+<wire x1="6.8678" y1="2.8284" x2="6.8678" y2="2.1492" width="0.1524" layer="1"/>
+<wire x1="6.8678" y1="2.1492" x2="7.366" y2="1.651" width="0.1524" layer="1"/>
+<wire x1="7.366" y1="1.651" x2="7.366" y2="0.381" width="0.1524" layer="1"/>
+<wire x1="7.366" y1="0.381" x2="7.239" y2="0.254" width="0.1524" layer="1"/>
+<wire x1="4.445" y1="0.254" x2="6.223" y2="0.254" width="0.1524" layer="1"/>
+<wire x1="6.223" y1="0.254" x2="7.239" y2="0.254" width="0.1524" layer="1"/>
+<wire x1="6.2178" y1="0.7784" x2="6.223" y2="0.7732" width="0.1524" layer="1"/>
+<wire x1="6.223" y1="0.7732" x2="6.223" y2="0.254" width="0.1524" layer="1"/>
 </signal>
 <signal name="12">
