File: cc2652r_v2_rs.sch (EAGLE design)
At the start: 56 parts, among them IC3 CC2652R1FRGZ, SW1 MOMENTARY-SWITCH-SPST-SMD-4.6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, Y1 Q22FA12800150, Y2 32.768KHz

Commit message: Add files via upload
Parts:
- removed C20, C22: CAP0402, discretes-dev:CAP0402
Connections:
- net 2: now also R3.1, REEDSWITCH.1; no longer R3.2, REEDSWITCH.2
- net GND: now also REEDSWITCH.2; no longer C20.1, C22.2, R3.1
- net VCC: now also R3.2; no longer REEDSWITCH.1
- net X48M_N: no longer C22.1
- net X48M_P: no longer C20.2
Other:
- moved on the sheet: R3, REEDSWITCH
Changed lines of the file:
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@@
 <part name="L5" library="discretes-dev" deviceset="IND0402" device="IND0402" value="2nH"/>
 <part name="L6" library="discretes-dev" deviceset="IND0402" device="IND0402" value="2nH"/>
-<part name="C20" library="discretes-dev" deviceset="CAP0402" device=""/>
-<part name="C22" library="discretes-dev" deviceset="CAP0402" device=""/>
-<part name="GND6" library="supply1" library_urn="urn:adsk.eagle:library:371" deviceset="GND" device=""/>
-<part name="GND20" library="supply1" library_urn="urn:adsk.eagle:library:371" deviceset="GND" device=""/>
 <part name="R2" library="discretes-dev" deviceset="RES0402" device="" value="2.2k"/>
 <part name="G" library="SparkFun-LED" library_urn="urn:adsk.eagle:library:529" deviceset="LED-GREEN" device="0603" package3d_urn="urn:adsk.eagle:package:39354/1" value="GREEN"/>
@@
 <attribute name="NAME" x="165.095559375" y="93.98148125" size="2.54148125" layer="95"/>
 </instance>
-<instance part="C20" gate="G$1" x="91.44" y="88.9" smashed="yes">
-<attribute name="NAME" x="92.964" y="90.551" size="1.778" layer="95" font="vector"/>
-</instance>
-<instance part="C22" gate="G$1" x="101.6" y="73.66" smashed="yes">
-<attribute name="NAME" x="103.124" y="75.311" size="1.778" layer="95" font="vector"/>
-</instance>
-<instance part="GND6" gate="1" x="101.6" y="66.04" smashed="yes">
-<attribute name="VALUE" x="99.06" y="63.5" size="1.778" layer="96"/>
-</instance>
-<instance part="GND20" gate="1" x="91.44" y="96.52" smashed="yes" rot="R180">
-<attribute name="VALUE" x="93.98" y="99.06" size="1.778" layer="96" rot="R180"/>
-</instance>
 <instance part="R2" gate="G$1" x="99.06" y="38.1" smashed="yes" rot="R90">
 <attribute name="NAME" x="96.51851875" y="30.475559375" size="2.54148125" layer="95" rot="R90"/>
@@
 <attribute name="VALUE" x="287.02" y="50.8" size="1.778" layer="96" rot="R180"/>
 </instance>
-<instance part="REEDSWITCH" gate="G$1" x="119.38" y="35.56" smashed="yes">
-<attribute name="NAME" x="121.92" y="38.1" size="1.778" layer="95"/>
+<instance part="REEDSWITCH" gate="G$1" x="119.38" y="17.78" smashed="yes">
+<attribute name="NAME" x="121.92" y="20.32" size="1.778" layer="95"/>
 </instance>
 <instance part="P+8" gate="VCC" x="119.38" y="50.8" smashed="yes">
 <attribute name="VALUE" x="116.84" y="48.26" size="1.778" layer="96" rot="R90"/>
 </instance>
-<instance part="R3" gate="G$1" x="119.38" y="20.32" smashed="yes" rot="R90">
-<attribute name="NAME" x="116.83851875" y="12.695559375" size="2.54148125" layer="95" rot="R90"/>
+<instance part="R3" gate="G$1" x="119.38" y="38.1" smashed="yes" rot="R90">
+<attribute name="NAME" x="116.83851875" y="30.475559375" size="2.54148125" layer="95" rot="R90"/>
 </instance>
 <instance part="GND30" gate="1" x="119.38" y="7.62" smashed="yes">
@@
 <pinref part="IC3" gate="G$1" pin="X48M_P"/>
 <wire x1="91.44" y1="81.28" x2="83.82" y2="81.28" width="0.1524" layer="91"/>
-<pinref part="C20" gate="G$1" pin="2"/>
-<wire x1="91.44" y1="85.09" x2="91.44" y2="81.28" width="0.1524" layer="91"/>
-<junction x="91.44" y="81.28"/>
 </segment>
 </net>
@@
 <pinref part="IC3" gate="G$1" pin="X48M_N"/>
 <wire x1="83.82" y1="83.82" x2="101.6" y2="83.82" width="0.1524" layer="91"/>
-<wire x1="101.6" y1="83.82" x2="101.6" y2="77.47" width="0.1524" layer="91"/>
 <pinref part="Y1" gate="G$1" pin="3"/>
 <wire x1="101.6" y1="78.74" x2="99.06" y2="78.74" width="0.1524" layer="91"/>
-<pinref part="C22" gate="G$1" pin="1"/>
-<wire x1="101.6" y1="78.74" x2="101.6" y2="77.47" width="0.1524" layer="91"/>
+<wire x1="101.6" y1="83.82" x2="101.6" y2="78.74" width="0.1524" layer="91"/>
 </segment>
 </net>
@@
 <wire x1="154.94" y1="80.01" x2="154.94" y2="76.2" width="0.1524" layer="91"/>
 <pinref part="GND5" gate="1" pin="GND"/>
-</segment>
-<segment>
-<pinref part="C22" gate="G$1" pin="2"/>
-<pinref part="GND6" gate="1" pin="GND"/>
-<wire x1="101.6" y1="69.85" x2="101.6" y2="68.58" width="0.1524" layer="91"/>
-</segment>
-<segment>
-<pinref part="C20" gate="G$1" pin="1"/>
-<pinref part="GND20" gate="1" pin="GND"/>
-<wire x1="91.44" y1="92.71" x2="91.44" y2="93.98" width="0.1524" layer="91"/>
 </segment>
 <segment>
@@
 </segment>
 <segment>
-<pinref part="GND30" gate="1" pin="GND"/>
-<wire x1="119.38" y1="10.16" x2="119.38" y2="11.43" width="0.1524" layer="91"/>
-<pinref part="R3" gate="G$1" pin="1"/>
-</segment>
-<segment>
 <pinref part="C26" gate="G$1" pin="1"/>
 <pinref part="GND31" gate="1" pin="GND"/>
 <wire x1="205.74" y1="80.01" x2="205.74" y2="76.2" width="0.1524" layer="91"/>
+</segment>
+<segment>
+<pinref part="REEDSWITCH" gate="G$1" pin="2"/>
+<pinref part="GND30" gate="1" pin="GND"/>
+<wire x1="119.38" y1="12.7" x2="119.38" y2="10.16" width="0.1524" layer="91"/>
 </segment>
 </net>
@@
 </segment>
 <segment>
-<pinref part="REEDSWITCH" gate="G$1" pin="1"/>
-<pinref part="P+8" gate="VCC" pin="VCC"/>
-<wire x1="119.38" y1="43.18" x2="119.38" y2="48.26" width="0.1524" layer="91"/>
-</segment>
-<segment>
 <pinref part="R5" gate="G$1" pin="2"/>
 <wire x1="251.46" y1="67.31" x2="251.46" y2="68.58" width="0.1524" layer="91"/>
@@
 <wire x1="259.08" y1="67.31" x2="259.08" y2="68.58" width="0.1524" layer="91"/>
 <pinref part="P+10" gate="VCC" pin="VCC"/>
+</segment>
+<segment>
+<pinref part="P+8" gate="VCC" pin="VCC"/>
+<pinref part="R3" gate="G$1" pin="2"/>
+<wire x1="119.38" y1="48.26" x2="119.38" y2="46.99" width="0.1524" layer="91"/>
 </segment>
 </net>
@@
 </segment>
 <segment>
-<pinref part="R3" gate="G$1" pin="2"/>
-<pinref part="REEDSWITCH" gate="G$1" pin="2"/>
-<wire x1="119.38" y1="29.21" x2="119.38" y2="30.48" width="0.1524" layer="91"/>
-<wire x1="119.38" y1="30.48" x2="124.46" y2="30.48" width="0.1524" layer="91"/>
-<junction x="119.38" y="30.48"/>
-<label x="124.46" y="30.48" size="1.778" layer="95"/>
+<pinref part="R3" gate="G$1" pin="1"/>
+<pinref part="REEDSWITCH" gate="G$1" pin="1"/>
+<wire x1="119.38" y1="29.21" x2="119.38" y2="27.94" width="0.1524" layer="91"/>
+<wire x1="119.38" y1="27.94" x2="119.38" y2="25.4" width="0.1524" layer="91"/>
+<wire x1="119.38" y1="27.94" x2="129.54" y2="27.94" width="0.1524" layer="91"/>
+<junction x="119.38" y="27.94"/>
+<label x="129.54" y="27.94" size="1.778" layer="95"/>
 </segment>
 </net>
@@
 </segment>
 </net>
+<net name="N$12" class="0">
+<segment>
+<wire x1="101.6" y1="69.85" x2="101.6" y2="68.58" width="0.1524" layer="91"/>
+</segment>
+</net>

Commit message: Add files via upload
Connections:
- net 11: now also BME280.CSB, BME280.VDD, BME280.VDDIO, C24.2, C25.1, HTU21.VDD
- net VCC: no longer BME280.CSB, BME280.VDD, BME280.VDDIO, C24.2, C25.1, HTU21.VDD
Changed lines of the file:
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@@
 <part name="HTU21" library="HTU21D" deviceset="HTU21D" device=""/>
 <part name="GND25" library="supply1" library_urn="urn:adsk.eagle:library:371" deviceset="GND" device=""/>
-<part name="P+7" library="supply1" library_urn="urn:adsk.eagle:library:371" deviceset="VCC" device=""/>
 <part name="C24" library="ok-discretes-dev" deviceset="CAP" device="-0402" value="100n"/>
 <part name="BME280" library="bosch-bme280" deviceset="BME280" device=""/>
@@
 <attribute name="VALUE" x="274.32" y="12.7" size="1.778" layer="96"/>
 </instance>
-<instance part="P+7" gate="VCC" x="276.86" y="48.26" smashed="yes">
-<attribute name="VALUE" x="274.32" y="45.72" size="1.778" layer="96" rot="R90"/>
-</instance>
 <instance part="C24" gate="A" x="274.32" y="27.94" smashed="yes" rot="R90">
 <attribute name="NAME" x="278.003" y="28.4226" size="1.778" layer="95"/>
@@
 </segment>
 <segment>
-<pinref part="HTU21" gate="G$1" pin="VDD"/>
-<wire x1="269.24" y1="35.56" x2="274.32" y2="35.56" width="0.1524" layer="91"/>
-<wire x1="274.32" y1="35.56" x2="276.86" y2="35.56" width="0.1524" layer="91"/>
-<wire x1="276.86" y1="35.56" x2="276.86" y2="45.72" width="0.1524" layer="91"/>
-<pinref part="P+7" gate="VCC" pin="VCC"/>
-<pinref part="C24" gate="A" pin="2"/>
-<wire x1="274.32" y1="35.56" x2="274.32" y2="30.48" width="0.1524" layer="91"/>
-<junction x="274.32" y="35.56"/>
-<pinref part="BME280" gate="G$1" pin="CSB"/>
-<wire x1="287.02" y1="30.48" x2="284.48" y2="30.48" width="0.1524" layer="91"/>
-<wire x1="284.48" y1="30.48" x2="284.48" y2="35.56" width="0.1524" layer="91"/>
-<pinref part="BME280" gate="G$1" pin="VDD"/>
-<wire x1="284.48" y1="35.56" x2="287.02" y2="35.56" width="0.1524" layer="91"/>
-<wire x1="284.48" y1="35.56" x2="276.86" y2="35.56" width="0.1524" layer="91"/>
-<junction x="284.48" y="35.56"/>
-<junction x="276.86" y="35.56"/>
-<pinref part="BME280" gate="G$1" pin="VDDIO"/>
-<wire x1="312.42" y1="33.02" x2="314.96" y2="33.02" width="0.1524" layer="91"/>
-<wire x1="314.96" y1="33.02" x2="314.96" y2="40.64" width="0.1524" layer="91"/>
-<wire x1="314.96" y1="40.64" x2="284.48" y2="40.64" width="0.1524" layer="91"/>
-<wire x1="284.48" y1="40.64" x2="284.48" y2="35.56" width="0.1524" layer="91"/>
-<pinref part="C25" gate="A" pin="1"/>
-<junction x="284.48" y="40.64"/>
-</segment>
-<segment>
 <pinref part="R5" gate="G$1" pin="2"/>
 <wire x1="251.46" y1="67.31" x2="251.46" y2="68.58" width="0.1524" layer="91"/>
@@
 <label x="35.56" y="45.72" size="1.778" layer="95"/>
 </segment>
-</net>
+<segment>
+<pinref part="HTU21" gate="G$1" pin="VDD"/>
+<wire x1="269.24" y1="35.56" x2="274.32" y2="35.56" width="0.1524" layer="91"/>
+<pinref part="C24" gate="A" pin="2"/>
+<wire x1="274.32" y1="35.56" x2="274.32" y2="30.48" width="0.1524" layer="91"/>
+<junction x="274.32" y="35.56"/>
+<pinref part="BME280" gate="G$1" pin="CSB"/>
+<wire x1="287.02" y1="30.48" x2="284.48" y2="30.48" width="0.1524" layer="91"/>
+<wire x1="284.48" y1="30.48" x2="284.48" y2="35.56" width="0.1524" layer="91"/>
+<pinref part="BME280" gate="G$1" pin="VDD"/>
+<wire x1="284.48" y1="35.56" x2="287.02" y2="35.56" width="0.1524" layer="91"/>
+<wire x1="284.48" y1="35.56" x2="274.32" y2="35.56" width="0.1524" layer="91"/>
+<junction x="284.48" y="35.56"/>
+<pinref part="BME280" gate="G$1" pin="VDDIO"/>
+<wire x1="312.42" y1="33.02" x2="314.96" y2="33.02" width="0.1524" layer="91"/>
+<wire x1="314.96" y1="33.02" x2="314.96" y2="40.64" width="0.1524" layer="91"/>
+<wire x1="314.96" y1="40.64" x2="284.48" y2="40.64" width="0.1524" layer="91"/>
+<wire x1="284.48" y1="40.64" x2="284.48" y2="35.56" width="0.1524" layer="91"/>
+<pinref part="C25" gate="A" pin="1"/>
+<junction x="284.48" y="40.64"/>
+<wire x1="274.32" y1="35.56" x2="274.32" y2="48.26" width="0.1524" layer="91"/>
+<label x="274.32" y="45.72" size="1.778" layer="95"/>
+</segment>
+</net>
