File: v2.1/cc2652r_v2.1_rs.brd (EAGLE design)
At the start: 29.3 x 29.3 mm, 55 parts, among them IC3 CC2652R1FRGZ, Q1 SI2323DS, Q2 SI2323DS, SW1 MOMENTARY-SWITCH-SPST-SMD-4.6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, Y1 Q22FA12800150, Y2 32.768KHz

Commit message: Add files via upload
Parts:
- moved C3 0.48 mm to (17.3, 13.4)
- moved L4 0.47 mm to (17.3, 10.3)
- moved C4 0.45 mm to (17.3, 9.25)
Routing:
- net N$6: track 30.8 -> 31.7 mm
- net GND: vias 322 -> 327

Commit message: Add files via upload
Parts:
- moved Y1 0.50 mm to (13.7, 8.15)
Routing:
- net GND: track 25.0 -> 23.2 mm, vias 327 -> 335
- net X48M_P: track 4.94 -> 4.37 mm
- net VCC: vias 7 -> 8

Commit message: Add files via upload
Parts:
- C23: value 220uf -> 220uF; device Capacitor:CAPM7343X310 -> SparkFun-Capacitors:EIA3528
- moved C23 3.21 mm to (13.1, 24.2), turned to 90 degrees
- moved Q2 0.91 mm to (16.7, 24.8)
- moved Q1 0.90 mm to (20.1, 24.8)
- moved R5 0.63 mm to (5.52, 6.50)
- moved R6 0.63 mm to (6.69, 6.50)
- moved HTU21 0.51 mm to (2.64, 6.13)
- moved REEDSWITCH 0.30 mm to (17.3, 1.95)
- moved BME280 0.26 mm to (5.92, 2.06)
- moved TP1 0.20 mm to (23.8, 11.9)
- moved E1 0.12 mm to (24.0, 8.75)
- moved C21 0.11 mm to (22.6, 11.9)
- moved C19 0.11 mm to (21.7, 12.8)
- moved TCK 0.10 mm to (1.03, 23.7)
- moved GND 0.10 mm to (1.02, 18.6)
- moved TDI 0.10 mm to (1.04, 21.2)
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Connections:
- net GND: now also C23.C; no longer C23.2
- net VCC: now also C23.A; no longer C23.1
Routing:
- net N$8: track 14.8 -> 8.57 mm
- net 4: track 31.7 -> 30.8 mm
- net GND: track 23.2 -> 22.4 mm, vias 335 -> 328
- net 5: track 27.8 -> 27.2 mm
- net 11: track 46.7 -> 46.0 mm
Other:
- board size 29.3 x 29.3 mm -> 29 x 29 mm
