File: v2.1/cc2652r_v2.1_rs.sch (EAGLE design)
At the start: 55 parts, among them IC3 CC2652R1FRGZ, Q1 SI2323DS, Q2 SI2323DS, SW1 MOMENTARY-SWITCH-SPST-SMD-4.6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, Y1 Q22FA12800150, Y2 32.768KHz

Commit message: Add files via upload
Parts:
- C23: value 220uf -> 220uF; device Capacitor:C_TANTALUM-2917(7343-METRIC) -> SparkFun-Capacitors:68UF-POLAR-EIA3528-10V-10%(TANT)
Connections:
- net GND: now also C23.-; no longer C23.2
- net VCC: now also C23.+; no longer C23.1
Changed lines of the file:
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@@
 <part name="TP2" library="testpad" deviceset="TPSQ" device="TP15SQ" package3d_urn="urn:adsk.eagle:package:27975/1" value="TPSQTP15SQ"/>
 <part name="BT1" library="Batteries" deviceset="BATTERY" device="-20MM_SMD" package3d_urn="urn:adsk.eagle:package:37215/1"/>
-<part name="C23" library="Capacitor" library_urn="urn:adsk.eagle:library:16290819" deviceset="C" device="TANTALUM-2917(7343-METRIC)" package3d_urn="urn:adsk.eagle:package:16290891/2" technology="_" value="220uf"/>
+<part name="C23" library="SparkFun-Capacitors" library_urn="urn:adsk.eagle:library:510" deviceset="68UF-POLAR" device="-EIA3528-10V-10%(TANT)" package3d_urn="urn:adsk.eagle:package:37411/1" value="220uF"/>
 <part name="P+5" library="supply1" library_urn="urn:adsk.eagle:library:371" deviceset="VCC" device=""/>
 <part name="GND24" library="supply1" library_urn="urn:adsk.eagle:library:371" deviceset="GND" device=""/>
@@
 </segment>
 <segment>
-<pinref part="C23" gate="G$1" pin="2"/>
+<pinref part="C23" gate="G$1" pin="-"/>
 <pinref part="GND24" gate="1" pin="GND"/>
 </segment>
@@
 <segment>
 <pinref part="P+5" gate="VCC" pin="VCC"/>
-<pinref part="C23" gate="G$1" pin="1"/>
+<pinref part="C23" gate="G$1" pin="+"/>
 <wire x1="226.06" y1="27.94" x2="226.06" y2="25.4" width="0.1524" layer="91"/>
 </segment>
